Commit message: working cup and ball

File: urdf/chain.urdf.xacro (robot description, xacro)
@@ -140,5 +140,5 @@
 				<origin xyz="0 0 0"/>
 				<geometry>
-					<mesh filename="file://../meshes/cup1e-3.dae"/>
+					<mesh filename="package://cup_and_ball/meshes/cup1e-3.dae"/>
 				</geometry>
 				<max_contacts>10</max_contacts>
@@ -159,5 +159,5 @@
 				<origin xyz="0 0 0" />
 				<geometry>
-					<mesh filename="file://../meshes/cup1e-3.dae"/>
+					<mesh filename="package://cup_and_ball/meshes/cup1e-3.dae"/>
 				</geometry>
 			</visual>

Commit message: added gz launch

File: urdf/chain.urdf.xacro (robot description, xacro)
@@ -60,15 +60,4 @@
 			<dynamics damping="${chain_link_damping}" friction="${chain_link_friction}"/>
 		</joint>
-		<!-- <link name="${name}_junta3">
-			<inertial>
-			<mass value="0.0001" />
-			<inertia ixx="5.8083e-5" ixy="0" ixz="0" iyy="3.0833e-6" iyz="0" izz="5.9083e-5" />
-			</inertial>
-		</link>
-		<joint name="${name}_jointfixed" type="continuous">
-			<parent link="${name}_junta3"/>
-			<child link="${name}"/>
-			<axis xys="0 1 0"/>
-		</joint> -->
 	</xacro:macro>
 	<material name="Grey">
@@ -140,5 +129,5 @@
 				<origin xyz="0 0 0"/>
 				<geometry>
-					<mesh filename="package://cup_and_ball/meshes/cup1e-3.dae"/>
+					<mesh filename="package://cup_and_ball/meshes/cup1e-4.dae"/>
 				</geometry>
 				<max_contacts>10</max_contacts>
@@ -159,5 +148,5 @@
 				<origin xyz="0 0 0" />
 				<geometry>
-					<mesh filename="package://cup_and_ball/meshes/cup1e-3.dae"/>
+					<mesh filename="package://cup_and_ball/meshes/cup1e-4.dae"/>
 				</geometry>
 			</visual>
@@ -177,14 +166,14 @@
 	<xacro:link_gazebo name="cup"/>
 	<xacro:chain_link name="0" X="${link_length}" Y="${link_yz}" Z="${link_yz}" mass="0.001"/>
-	<!-- <xacro:link_ball_joint name="0" X="${link_length}" parent="dummy"/> -->
-	<joint name="chain_fixed" type="continuous">
+	<xacro:link_ball_joint name="0" X="${link_length}" parent="cup"/>
+	<!-- <joint name="chain_fixed" type="continuous">
 		<origin xyz="0 0 0" rpy="0 0 0" />
 		<parent link="cup"/>
 		<child link="0"/>
-	</joint>
+	</joint> -->
 	<xacro:link_gazebo name="0" />
 	<xacro:chain_loop i="${link_num}" />
-	<!-- <xacro:ball d="0.05" mass="1"/>
+	<xacro:ball d="0.05" mass="1"/>
 	<xacro:link_gazebo name="ball"/>
-	<xacro:link_ball_joint name="ball" X="${link_length}" parent="${link_num}"/> -->
+	<xacro:link_ball_joint name="ball" X="${link_length}" parent="${link_num}"/>
 </robot>

Commit message: working model except physics

File: urdf/chain.urdf.xacro (robot description, xacro)
@@ -34,5 +34,5 @@
 			<child link="${name}_phi"/>
 			<axis xyz="1 0 0" />
-			<dynamics damping="${chain_link_damping}" friction="${chain_link_friction}"/>
+			<!-- <dynamics damping="${chain_link_damping}" friction="${chain_link_friction}"/> -->
 		</joint>
 		<link name="${name}_phi">
@@ -46,5 +46,5 @@
 			<child link="${name}_psi"/>
 			<axis xyz="0 1 0" />
-			<dynamics damping="${chain_link_damping}" friction="${chain_link_friction}"/>
+			<!-- <dynamics damping="${chain_link_damping}" friction="${chain_link_friction}"/> -->
 		</joint>
 		<link name="${name}_psi">
@@ -58,5 +58,5 @@
 			<child link="${name}"/>
 			<axis xyz="0 0 1" />
-			<dynamics damping="${chain_link_damping}" friction="${chain_link_friction}"/>
+			<!-- <dynamics damping="${chain_link_damping}" friction="${chain_link_friction}"/> -->
 		</joint>
 	</xacro:macro>
@@ -64,18 +64,31 @@
 		<color rgba="0.7 0.7 0.7 1.0"/>
 	</material>
+	<xacro:macro name="link_gazebo_chain" params="name">
+		<gazebo reference="${name}">
+			<selfCollide>false</selfCollide>
+			<!--dampingFactor>0.0001</dampingFactor-->
+			<material>Grey</material>
+		</gazebo>
+		<gazebo reference="${name}_x">
+			<implicitSpringDamper>true</implicitSpringDamper>
+		</gazebo>
+		<gazebo reference="${name}_y">
+			<implicitSpringDamper>true</implicitSpringDamper>
+		</gazebo>
+		<gazebo reference="${name}_z">
+			<implicitSpringDamper>true</implicitSpringDamper>
+		</gazebo>
+	</xacro:macro>
 	<xacro:macro name="link_gazebo" params="name">
-	  <gazebo reference="${name}">
-		  <selfCollide>false</selfCollide>
-		  <!--dampingFactor>0.0001</dampingFactor-->
-		  <material>Grey</material>
-	  </gazebo>
-	  <gazebo reference="${name}_link_joint">
-		  <implicitSpringDamper>true</implicitSpringDamper>
-	  </gazebo>
+		<gazebo reference="${name}">
+			<selfCollide>false</selfCollide>
+			<!--dampingFactor>0.0001</dampingFactor-->
+			<material>Grey</material>
+		</gazebo>
 	</xacro:macro>
 	<xacro:macro name="chain_loop" params="i">
 		<xacro:chain_link name="${link_num - i + 1}" X="${link_length}" Y="${link_yz}" Z="${link_yz}" mass="${chain_link_mass}"/>
 		<xacro:link_ball_joint name="${link_num - i + 1}" X="${link_length}" parent="${link_num - i}"/>
-		<xacro:link_gazebo name="${link_num - i + 1}"/>
+		<xacro:link_gazebo_chain name="${link_num - i + 1}"/>
 		<xacro:if value="${i-1}">
 			<xacro:chain_loop i="${i-1}" />
@@ -117,17 +130,17 @@
 			<enable_wind>0</enable_wind>
 			<kinematic>0</kinematic>
-	  	</link>
+		</link>
 	</xacro:macro>
 	<xacro:macro name="cup" params="mass">
 		<link name="cup">
 			<inertial>
-				<origin xyz="0 0 0" />
+				<origin xyz="-0.01 -0.25 0"/>
 				<mass value="${mass}"/>
 				<inertia ixx="${mass * 0.282601}" ixy="${mass * 0.0056}" ixz="${mass * -0.000002}" iyy="${mass * 0.147524}" iyz="${mass * -0.007428}" izz="${mass * 0.276385}"/>
 			</inertial>
 			<collision name='collision'>
-				<origin xyz="0 0 0"/>
+				<origin xyz="-0.01 -0.25 0"/>
 				<geometry>
-					<mesh filename="package://cup_and_ball/meshes/cup1e-4.dae"/>
+					<mesh filename="package://cup_and_ball/meshes/cup.dae" scale="0.001 0.001 0.001"/>
 				</geometry>
 				<max_contacts>10</max_contacts>
@@ -146,7 +159,7 @@
 			</collision>
 			<visual name='visual'>
-				<origin xyz="0 0 0" />
+				<origin xyz="-0.01 -0.25 0"/>
 				<geometry>
-					<mesh filename="package://cup_and_ball/meshes/cup1e-4.dae"/>
+					<mesh filename="package://cup_and_ball/meshes/cup.dae" scale="0.001 0.001 0.001"/>
 				</geometry>
 			</visual>
@@ -154,5 +167,5 @@
 			<enable_wind>0</enable_wind>
 			<kinematic>0</kinematic>
-	  	</link>
+		</link>
 	</xacro:macro>
 	<!-- build chain links with base at the bottom usign the loop. build ball, attach to chain -->
@@ -166,14 +179,14 @@
 	<xacro:link_gazebo name="cup"/>
 	<xacro:chain_link name="0" X="${link_length}" Y="${link_yz}" Z="${link_yz}" mass="0.001"/>
-	<xacro:link_ball_joint name="0" X="${link_length}" parent="cup"/>
-	<!-- <joint name="chain_fixed" type="continuous">
+	<!-- <xacro:link_ball_joint name="0" X="${link_length}" parent="cup"/> -->
+	<joint name="chain_fixed" type="continuous">
 		<origin xyz="0 0 0" rpy="0 0 0" />
 		<parent link="cup"/>
 		<child link="0"/>
-	</joint> -->
+	</joint>
 	<xacro:link_gazebo name="0" />
 	<xacro:chain_loop i="${link_num}" />
 	<xacro:ball d="0.05" mass="1"/>
-	<xacro:link_gazebo name="ball"/>
+	<xacro:link_gazebo_chain name="ball"/>
 	<xacro:link_ball_joint name="ball" X="${link_length}" parent="${link_num}"/>
 </robot>

Commit message: two dof ball joint

File: urdf/chain.urdf.xacro (robot description, xacro)
@@ -1,10 +1,10 @@
 <?xml version="1.0"?>
 <robot xmlns:xacro="http://www.ros.org/wiki/xacro" name="chain">
-	<xacro:property name="link_length" value="0.025" />
+	<xacro:property name="link_length" value="0.075" />
 	<xacro:property name="link_yz" value="0.001"/>
-	<xacro:property name="link_num" value="20"/>
-	<xacro:property name="chain_link_mass" value="0.0001"/>
-	<xacro:property name="chain_link_damping" value="1.0"/>
-	<xacro:property name="chain_link_friction" value="1.0"/>
+	<xacro:property name="link_num" value="4"/>
+	<xacro:property name="chain_link_mass" value="0.001"/>
+	<xacro:property name="chain_link_damping" value="100.0"/>
+	<xacro:property name="chain_link_friction" value="0.0"/>
 	<xacro:macro name="chain_link" params="name X Y Z mass">
 		<link name="${name}">
@@ -33,6 +33,39 @@
 			<parent link="${parent}"/>
 			<child link="${name}_phi"/>
+			<axis xyz="0 1 0" />
+			<dynamics damping="${chain_link_damping}" friction="${chain_link_friction}"/>
+		</joint>
+		<link name="${name}_phi">
+			<inertial>
+				<mass value="0.0001" />
+				<inertia ixx="5.8083e-5" ixy="0" ixz="0" iyy="3.0833e-6" iyz="0" izz="5.9083e-5" />
+			</inertial>
+		</link>
+		<joint name="${name}_y" type="continuous">
+			<parent link="${name}_phi"/>
+			<child link="${name}"/>
+			<axis xyz="0 0 1" />
+			<dynamics damping="${chain_link_damping}" friction="${chain_link_friction}"/>
+		</joint>
+		<!-- <link name="${name}_psi">
+			<inertial>
+				<mass value="0.0001" />
+				<inertia ixx="5.8083e-5" ixy="0" ixz="0" iyy="3.0833e-6" iyz="0" izz="5.9083e-5" />
+			</inertial>
+		</link>
+		<joint name="${name}_z" type="continuous">
+			<parent link="${name}_psi"/>
+			<child link="${name}"/>
 			<axis xyz="1 0 0" />
-			<!-- <dynamics damping="${chain_link_damping}" friction="${chain_link_friction}"/> -->
+			<dynamics damping="${chain_link_damping}" friction="${chain_link_friction}"/>
+		</joint> -->
+	</xacro:macro>
+	<xacro:macro name="link_ball_joint_ball" params="name X parent">
+		<joint name="${name}_x" type="continuous">
+			<origin xyz="${X} 0 0" rpy="0 0 0"/>
+			<parent link="${parent}"/>
+			<child link="${name}_phi"/>
+			<axis xyz="1 0 0" />
+			<dynamics damping="${chain_link_damping}" friction="${chain_link_friction}"/>
 		</joint>
 		<link name="${name}_phi">
@@ -46,5 +79,5 @@
 			<child link="${name}_psi"/>
 			<axis xyz="0 1 0" />
-			<!-- <dynamics damping="${chain_link_damping}" friction="${chain_link_friction}"/> -->
+			<dynamics damping="${chain_link_damping}" friction="${chain_link_friction}"/>
 		</joint>
 		<link name="${name}_psi">
@@ -58,5 +91,4 @@
 			<child link="${name}"/>
 			<axis xyz="0 0 1" />
-			<!-- <dynamics damping="${chain_link_damping}" friction="${chain_link_friction}"/> -->
 		</joint>
 	</xacro:macro>
@@ -80,7 +112,23 @@
 		</gazebo>
 	</xacro:macro>
+	<xacro:macro name="link_gazebo_chain_self_collide" params="name">
+		<gazebo reference="${name}">
+			<selfCollide>true</selfCollide>
+			<!--dampingFactor>0.0001</dampingFactor-->
+			<material>Grey</material>
+		</gazebo>
+		<gazebo reference="${name}_x">
+			<implicitSpringDamper>true</implicitSpringDamper>
+		</gazebo>
+		<gazebo reference="${name}_y">
+			<implicitSpringDamper>true</implicitSpringDamper>
+		</gazebo>
+		<gazebo reference="${name}_z">
+			<implicitSpringDamper>true</implicitSpringDamper>
+		</gazebo>
+	</xacro:macro>
 	<xacro:macro name="link_gazebo" params="name">
 		<gazebo reference="${name}">
-			<selfCollide>false</selfCollide>
+			<selfCollide>true</selfCollide>
 			<!--dampingFactor>0.0001</dampingFactor-->
 			<material>Grey</material>
@@ -135,7 +183,12 @@
 		<link name="cup">
 			<inertial>
-				<origin xyz="-0.01 -0.25 0"/>
+				<origin xyz="-0.01 0 0"/>
 				<mass value="${mass}"/>
-				<inertia ixx="${mass * 0.282601}" ixy="${mass * 0.0056}" ixz="${mass * -0.000002}" iyy="${mass * 0.147524}" iyz="${mass * -0.007428}" izz="${mass * 0.276385}"/>
+				<inertia 	ixx="${mass * -0.333449}"
+							ixy="${mass * 0.0}"
+							ixz="${mass * -0.000074}"
+							iyy="${mass * -0.333453}"
+							iyz="${mass * -0.000001}"
+							izz="${mass * -0.125942}"/>
 			</inertial>
 			<collision name='collision'>
@@ -188,5 +241,5 @@
 	<xacro:chain_loop i="${link_num}" />
 	<xacro:ball d="0.05" mass="1"/>
-	<xacro:link_gazebo_chain name="ball"/>
-	<xacro:link_ball_joint name="ball" X="${link_length}" parent="${link_num}"/>
+	<xacro:link_gazebo_chain_self_collide name="ball"/>
+	<xacro:link_ball_joint_ball name="ball" X="${link_length}" parent="${link_num}"/>
 </robot>

Commit message: roll pitch yaw control

File: urdf/chain.urdf.xacro (robot description, xacro)
@@ -1,7 +1,7 @@
 <?xml version="1.0"?>
 <robot xmlns:xacro="http://www.ros.org/wiki/xacro" name="chain">
-	<xacro:property name="link_length" value="0.075" />
+	<xacro:property name="link_length" value="0.06" />
 	<xacro:property name="link_yz" value="0.001"/>
-	<xacro:property name="link_num" value="4"/>
+	<xacro:property name="link_num" value="5"/>
 	<xacro:property name="chain_link_mass" value="0.001"/>
 	<xacro:property name="chain_link_damping" value="100.0"/>
@@ -66,5 +66,5 @@
 			<parent link="${parent}"/>
 			<child link="${name}_phi"/>
-			<axis xyz="1 0 0" />
+			<axis xyz="0 1 0" />
 			<dynamics damping="${chain_link_damping}" friction="${chain_link_friction}"/>
 		</joint>
@@ -78,5 +78,5 @@
 			<parent link="${name}_phi"/>
 			<child link="${name}_psi"/>
-			<axis xyz="0 1 0" />
+			<axis xyz="0 0 1" />
 			<dynamics damping="${chain_link_damping}" friction="${chain_link_friction}"/>
 		</joint>
@@ -90,5 +90,5 @@
 			<parent link="${name}_psi"/>
 			<child link="${name}"/>
-			<axis xyz="0 0 1" />
+			<axis xyz="1 0 0" />
 		</joint>
 	</xacro:macro>

Commit message: fixed majority of physics issues

File: urdf/chain.urdf.xacro (robot description, xacro)
@@ -1,9 +1,9 @@
 <?xml version="1.0"?>
 <robot xmlns:xacro="http://www.ros.org/wiki/xacro" name="chain">
-	<xacro:property name="link_length" value="0.06" />
-	<xacro:property name="link_yz" value="0.001"/>
-	<xacro:property name="link_num" value="5"/>
-	<xacro:property name="chain_link_mass" value="0.001"/>
-	<xacro:property name="chain_link_damping" value="100.0"/>
+	<xacro:property name="link_length" value="0.03" />
+	<xacro:property name="link_yz" value="0.005"/>
+	<xacro:property name="link_num" value="10"/>
+	<xacro:property name="chain_link_mass" value="0.025"/>
+	<xacro:property name="chain_link_damping" value="1.0"/>
 	<xacro:property name="chain_link_friction" value="0.0"/>
 	<xacro:macro name="chain_link" params="name X Y Z mass">
@@ -224,5 +224,5 @@
 	<!-- build chain links with base at the bottom usign the loop. build ball, attach to chain -->
 	<link name="base_link"/>
-	<xacro:cup mass="1"/>
+	<xacro:cup mass=".25"/>
 	<joint name="cup_fixed" type="fixed">
 		<origin xyz="0 0 0" rpy="0 0 0" />
@@ -240,5 +240,5 @@
 	<xacro:link_gazebo name="0" />
 	<xacro:chain_loop i="${link_num}" />
-	<xacro:ball d="0.05" mass="1"/>
+	<xacro:ball d="0.05" mass=".1"/>
 	<xacro:link_gazebo_chain_self_collide name="ball"/>
 	<xacro:link_ball_joint_ball name="ball" X="${link_length}" parent="${link_num}"/>

Commit message: testing new interia matrices

File: urdf/chain.urdf.xacro (robot description, xacro)
@@ -1,8 +1,8 @@
 <?xml version="1.0"?>
 <robot xmlns:xacro="http://www.ros.org/wiki/xacro" name="chain">
-	<xacro:property name="link_length" value="0.03" />
+	<xacro:property name="link_length" value="0.025" />
 	<xacro:property name="link_yz" value="0.005"/>
 	<xacro:property name="link_num" value="10"/>
-	<xacro:property name="chain_link_mass" value="0.025"/>
+	<xacro:property name="chain_link_mass" value="0.015"/>
 	<xacro:property name="chain_link_damping" value="1.0"/>
 	<xacro:property name="chain_link_friction" value="0.0"/>
@@ -24,5 +24,5 @@
 				<origin xyz="${X/2} 0 0" rpy="0 0 0" />
 				<mass value="${mass}"/>
-				<inertia ixx="${mass*(Y*Y + Z*Z)/12}" ixy="0.00" ixz="0.00" iyy="${mass*(X*X + Z*Z)/12}" iyz="0.00" izz="${mass*(X*X + Y*Y)/12}"/>
+				<inertia ixx="${mass*(Y*Y + Z*Z)/12}" ixy="0.00" ixz="0.00" iyy="${mass*(X*X + Z*Z)/12}" iyz="0.00" izz="${mass*(Y*Y + Z*Z)/12}"/>
 			</inertial>
 		</link>
@@ -39,5 +39,5 @@
 			<inertial>
 				<mass value="0.0001" />
-				<inertia ixx="5.8083e-5" ixy="0" ixz="0" iyy="3.0833e-6" iyz="0" izz="5.9083e-5" />
+				<inertia ixx="5.8083e-5" ixy="0" ixz="0" iyy="5.8083e-5" iyz="0" izz="5.8083e-5" />
 			</inertial>
 		</link>
@@ -72,5 +72,5 @@
 			<inertial>
 				<mass value="0.0001" />
-				<inertia ixx="5.8083e-5" ixy="0" ixz="0" iyy="3.0833e-6" iyz="0" izz="5.9083e-5" />
+				<inertia ixx="5.8083e-5" ixy="0" ixz="0" iyy="5.8083e-5" iyz="0" izz="5.8083e-5" />
 			</inertial>
 		</link>
@@ -84,5 +84,5 @@
 			<inertial>
 				<mass value="0.0001" />
-				<inertia ixx="5.8083e-5" ixy="0" ixz="0" iyy="3.0833e-6" iyz="0" izz="5.9083e-5" />
+				<inertia ixx="5.8083e-5" ixy="0" ixz="0" iyy="5.8083e-5" iyz="0" izz="5.8083e-5" />
 			</inertial>
 		</link>
